Commit message: Update URDF path and adjust joint parameters in spm_urdf_pybullet script

File: spm_wrist_description/urdf/spm_wrist.urdf (robot description, URDF)
Before this commit: robot spm_wrist, 25 links, 24 joints
Joints:
- joint world_joint: origin xyz=0.0 0.0 0.20 rpy=1.570796325 0.0 0.0 -> xyz=0.0 0.0 0.0 rpy=1.570796325 0.0 0.0
